Commit message: revert back to xmllint

File: examples/irb140/urdf/xacro/irb_140_robotiq.xacro (robot description, xacro)
@@ -1,5 +1,6 @@
+<?xml version="1.0"?>
 <robot xmlns:xacro="http://www.ros.org/wiki/xacro" name="IRB140">
-  <xacro:include filename="../irb_140.urdf" />
-  <xacro:include filename="../../../Atlas/urdf/robotiq.urdf" />
+  <xacro:include filename="../irb_140.urdf"/>
+  <xacro:include filename="../../../Atlas/urdf/robotiq.urdf"/>
   <joint name="robotiq_hand_joint" type="fixed">
     <origin rpy="0.0 0.0 -1.57079" xyz="0.11904 0 0"/>

File: examples/irb140/urdf/xacro/irb_140_robotiq_ati.xacro (robot description, xacro)
@@ -1,6 +1,7 @@
+<?xml version="1.0"?>
 <robot xmlns:xacro="http://www.ros.org/wiki/xacro" name="IRB140">
-  <xacro:include filename="../../../Atlas/urdf/robotiq.urdf" />
-  <xacro:include filename="../irb_140.urdf" />
-  <xacro:include filename="../ATI_sensor.urdf" />
+  <xacro:include filename="../../../Atlas/urdf/robotiq.urdf"/>
+  <xacro:include filename="../irb_140.urdf"/>
+  <xacro:include filename="../ATI_sensor.urdf"/>
   <joint name="robotiq_hand_joint" type="fixed">
     <origin rpy="0.0 0.0 -1.57079" xyz="0.11904 0 0"/>

File: examples/irb140/urdf/xacro/irb_140_robotiq_simple_ati.xacro (robot description, xacro)
@@ -1,6 +1,7 @@
+<?xml version="1.0"?>
 <robot xmlns:xacro="http://www.ros.org/wiki/xacro" name="IRB140">
-  <xacro:include filename="../../../Atlas/urdf/robotiq_simple.urdf" />
-  <xacro:include filename="../irb_140.urdf" />
-  <xacro:include filename="../ATI_sensor.urdf" />
+  <xacro:include filename="../../../Atlas/urdf/robotiq_simple.urdf"/>
+  <xacro:include filename="../irb_140.urdf"/>
+  <xacro:include filename="../ATI_sensor.urdf"/>
   <joint name="robotiq_hand_joint" type="fixed">
     <origin rpy="0.0 0.0 -1.57079" xyz="0.11904 0 0"/>

File: examples/planar_gripper/planar_gripper.xacro (robot description, xacro)
@@ -1,26 +1,26 @@
 <?xml version="1.0"?>
-<sdf xmlns:xacro="http://www.ros.org/wiki/xacro" version='1.7'>
-  <model name='planar_gripper'>
+<sdf xmlns:xacro="http://www.ros.org/wiki/xacro" version="1.6">
+  <model name="planar_gripper">
     <!-- Link mass and inertia values are guesses (currently), calculated using
          a uniform rod model, rotating about its center of mass. -->
-    <xacro:property name="base_dim" value=".08" />
-    <xacro:property name="l1_length" value="0.085" />
-    <xacro:property name="l1_radius" value="0.011" />
-    <xacro:property name="l1_mass" value="0.1" />
-    <xacro:property name="l1_inertia" value="0.0083" />
-    <xacro:property name="l2_length" value="0.040" />
-    <xacro:property name="l2_radius" value="0.011" />
-    <xacro:property name="l2_mass" value="0.1" />
-    <xacro:property name="l2_inertia" value="0.0083" />
-    <xacro:property name="sensor_length" value="0.005" />
-    <xacro:property name="sensor_width" value="0.02" />
-    <xacro:property name="tip_adapter_length" value="0.0113" />
-    <xacro:property name="tip_adapter_radius" value="0.0145" />
-    <xacro:property name="tip_cylinder_length" value="0.0035" />
-    <xacro:property name="tip_cylinder_radius" value="0.01" />
-    <xacro:property name="tip_sphere_radius" value="0.015" />
+    <xacro:property name="base_dim" value=".08"/>
+    <xacro:property name="l1_length" value="0.085"/>
+    <xacro:property name="l1_radius" value="0.011"/>
+    <xacro:property name="l1_mass" value="0.1"/>
+    <xacro:property name="l1_inertia" value="0.0083"/>
+    <xacro:property name="l2_length" value="0.040"/>
+    <xacro:property name="l2_radius" value="0.011"/>
+    <xacro:property name="l2_mass" value="0.1"/>
+    <xacro:property name="l2_inertia" value="0.0083"/>
+    <xacro:property name="sensor_length" value="0.005"/>
+    <xacro:property name="sensor_width" value="0.02"/>
+    <xacro:property name="tip_adapter_length" value="0.0113"/>
+    <xacro:property name="tip_adapter_radius" value="0.0145"/>
+    <xacro:property name="tip_cylinder_length" value="0.0035"/>
+    <xacro:property name="tip_cylinder_radius" value="0.01"/>
+    <xacro:property name="tip_sphere_radius" value="0.015"/>
     <xacro:macro name="finger" params="fnum">
       <link name="finger${fnum}_base">
-        <visual name='base_visual'>
+        <visual name="base_visual">
           <pose>0 0 0 0 0 0</pose>
           <geometry>
@@ -40,9 +40,13 @@
           <mass>${l1_mass}</mass>
           <inertia>
-            <ixx>${l1_inertia}</ixx><iyy>${l1_inertia}</iyy><izz>5e-7</izz>
-            <ixy>0</ixy><ixz>0</ixz><iyz>0</iyz>
+            <ixx>${l1_inertia}</ixx>
+            <iyy>${l1_inertia}</iyy>
+            <izz>5e-7</izz>
+            <ixy>0</ixy>
+            <ixz>0</ixz>
+            <iyz>0</iyz>
           </inertia>
         </inertial>
-        <visual name='link1_visual'>
+        <visual name="link1_visual">
           <pose>0 0 -${l1_length/2} 0 0 0</pose>
           <geometry>
@@ -56,5 +60,5 @@
           </material>
         </visual>
-        <visual name='link1_joint_visual'>
+        <visual name="link1_joint_visual">
           <pose>0 0 -${l1_length} 0 0 0</pose>
           <geometry>
@@ -68,5 +72,5 @@
         </visual>
       </link>
-      <joint name='finger${fnum}_BaseJoint' type='revolute'>
+      <joint name="finger${fnum}_BaseJoint" type="revolute">
         <child>finger${fnum}_link1</child>
         <parent>finger${fnum}_base</parent>
@@ -92,9 +96,13 @@
           <mass>${l2_mass}</mass>
           <inertia>
-            <ixx>${l2_inertia}</ixx><iyy>${l2_inertia}</iyy><izz>5e-7</izz>
-            <ixy>0</ixy><ixz>0</ixz><iyz>0</iyz>
+            <ixx>${l2_inertia}</ixx>
+            <iyy>${l2_inertia}</iyy>
+            <izz>5e-7</izz>
+            <ixy>0</ixy>
+            <ixz>0</ixz>
+            <iyz>0</iyz>
           </inertia>
         </inertial>
-        <visual name='link2_visual'>
+        <visual name="link2_visual">
           <pose>0 0 -${l2_length/2} 0 0 0</pose>
           <geometry>
@@ -110,5 +118,5 @@
         <!--The link 2 collision element extends up to (but not including) the
             sphere fingertip-->
-        <collision name='link2_collision'>
+        <collision name="link2_collision">
           <pose>0 0 -${(l2_length + sensor_length + tip_adapter_length + tip_cylinder_length)/2} 0 0 0</pose>
           <geometry>
@@ -121,5 +129,5 @@
           </material>
         </collision>
-        <visual name='sensor_visual'>
+        <visual name="sensor_visual">
           <pose>0 0 -${l2_length + sensor_length/2.0} 0 0 0</pose>
           <geometry>
@@ -133,5 +141,5 @@
         </visual>
       </link>
-      <joint name='finger${fnum}_MidJoint' type='revolute'>
+      <joint name="finger${fnum}_MidJoint" type="revolute">
         <parent>finger${fnum}_link1</parent>
         <child>finger${fnum}_link2</child>
@@ -162,6 +170,10 @@
           <mass>1e-7</mass>
           <inertia>
-            <ixx>1e-7</ixx><iyy>1e-7</iyy><izz>1e-7</izz>
-            <ixy>0</ixy><ixz>0</ixz><iyz>0</iyz>
+            <ixx>1e-7</ixx>
+            <iyy>1e-7</iyy>
+            <izz>1e-7</izz>
+            <ixy>0</ixy>
+            <ixz>0</ixz>
+            <iyz>0</iyz>
           </inertia>
         </inertial>
@@ -190,5 +202,5 @@
           </material>
         </visual>
-        <visual name='tip_sphere_visual'>
+        <visual name="tip_sphere_visual">
           <pose>0 0 -${tip_adapter_length + tip_sphere_radius} 0 0 0</pose>
           <geometry>
@@ -201,5 +213,5 @@
           </material>
         </visual>
-        <collision name='tip_sphere_collision'>
+        <collision name="tip_sphere_collision">
           <pose>0 0 -${tip_adapter_length + tip_sphere_radius} 0 0 0</pose>
           <geometry>
@@ -213,5 +225,5 @@
         </collision>
       </link>
-      <joint name='finger${fnum}_sensor_weldjoint' type='fixed'>
+      <joint name="finger${fnum}_sensor_weldjoint" type="fixed">
         <parent>finger${fnum}_link2</parent>
         <child>finger${fnum}_tip_link</child>
@@ -219,7 +231,7 @@
       </joint>
     </xacro:macro>
-    <xacro:finger fnum="1" />
-    <xacro:finger fnum="2" />
-    <xacro:finger fnum="3" />
+    <xacro:finger fnum="1"/>
+    <xacro:finger fnum="2"/>
+    <xacro:finger fnum="3"/>
   </model>
 </sdf>

File: manipulation/models/wsg_50_description/urdf/wsg_50.urdf.xacro (robot description, xacro)
@@ -13,5 +13,5 @@
   files in this directory.
 -->
-<robot name="wsg_50" xmlns:controller="http://playerstage.sourceforge.net/gazebo/xmlschema/#controller" xmlns:interface="http://playerstage.sourceforge.net/gazebo/xmlschema/#interface" xmlns:sensor="http://playerstage.sourceforge.net/gazebo/xmlschema/#sensor" xmlns:xacro="http://ros.org/wiki/xacro">
+<robot xmlns:controller="http://playerstage.sourceforge.net/gazebo/xmlschema/#controller" xmlns:interface="http://playerstage.sourceforge.net/gazebo/xmlschema/#interface" xmlns:sensor="http://playerstage.sourceforge.net/gazebo/xmlschema/#sensor" xmlns:xacro="http://ros.org/wiki/xacro" name="wsg_50">
   <xacro:macro name="wsg_50" params="name parent *origin">
     <joint name="${name}_anterior_gripper_joint" type="fixed">

File: manipulation/models/wsg_50_description/urdf/wsg_50_mesh_collision.urdf.xacro (robot description, xacro)
@@ -8,5 +8,5 @@
      macro automatically defaults to use mesh collision models.-->
 <!-- ===================================================================== -->
-<robot name="wsg_50" xmlns:xacro="http://www.ros.org/wiki/xacro">
+<robot xmlns:xacro="http://www.ros.org/wiki/xacro" name="wsg_50">
   <!-- Imports the wsg_50 macro. -->
   <xacro:include filename="$(find wsg_50_description)/urdf/wsg_50.urdf.xacro"/>
@@ -14,5 +14,5 @@
   <xacro:arg default="world" name="parent"/>
   <!-- Instantiates a WSG 50 URDF model by calling the wsg_50 macro. -->
-  <link name="world"></link>
+  <link name="world"/>
   <xacro:wsg_50 name="$(arg robot_name)" parent="$(arg parent)">
     <origin rpy="0 0 0" xyz="0 0 0"/>
