Commit message: fixup! add workflow test

File: multibody/benchmarks/free_body/uniform_solid_cylinder.urdf (robot description, URDF)
Before this commit: robot uniformSolidCylinderNoForceTorque, 1 links, 0 joints
Links:
- link uniformSolidCylinder: geometry collision cylinder length=0.6 radius=0.2; visual cylinder length=0.6 radius=0.2
